Commit message: Align wheel joint axes with robot coordinate convention

File: ros2_ws/src/robot_bringup/urdf/mobile_robot.urdf (robot description, URDF)
Before this commit: robot mobile_robot, 3 links, 2 joints
Joints:
- joint left_wheel_joint: axis 0 0 1 -> 0 1 0; origin xyz=0 0.2 0 rpy=1.5708 0 0 -> xyz=0 0.2 0 rpy=0 0 0
- joint right_wheel_joint: axis 0 0 1 -> 0 1 0; origin xyz=0 -0.2 0 rpy=1.5708 0 0 -> xyz=0 -0.2 0 rpy=0 0 0

Commit message: Add base footprint frame to mobile robot model

File: ros2_ws/src/robot_bringup/urdf/mobile_robot.urdf (robot description, URDF)
Before this commit: robot mobile_robot, 3 links, 2 joints
Links:
- added link base_footprint
Joints:
- added joint base_footprint_joint: type fixed, parent base_footprint, child base_link, origin xyz=0 0 0.125 rpy=0 0 0

Commit message: Add collision geometry to mobile robot model

File: ros2_ws/src/robot_bringup/urdf/mobile_robot.urdf (robot description, URDF)
Before this commit: robot mobile_robot, 4 links, 3 joints
Links:
- link base_link: geometry collision box size=0.6 0.4 0.15; visual box size=0.6 0.4 0.15
- link left_wheel_link: geometry collision cylinder length=0.04 radius=0.05; visual cylinder length=0.04 radius=0.05
- link right_wheel_link: geometry collision cylinder length=0.04 radius=0.05; visual cylinder length=0.04 radius=0.05

Commit message: Add inertial properties to mobile robot model

File: ros2_ws/src/robot_bringup/urdf/mobile_robot.urdf (robot description, URDF)
Before this commit: robot mobile_robot, 4 links, 3 joints
Links:
- link base_link: mass None -> 5.0
- link left_wheel_link: mass None -> 0.2
- link right_wheel_link: mass None -> 0.2
